Commit message: may 25 update

File: ackerman_ws/src/carmodel/urdf/car.xacro (robot description, xacro)
@@ -1,3 +1,2 @@
-<!-- 组合小车底盘与摄像头 -->
 <robot name="my_car_camera" xmlns:xacro="http://wiki.ros.org/xacro">
     <xacro:include filename="headfile.xacro" />

File: ackerman_ws/src/carmodel/urdf/smart.xacro (robot description, xacro)
@@ -2,4 +2,7 @@
 <robot name="$(arg roboname)" xmlns:xacro="http://www.ros.org/wiki/xacro">
   <xacro:property name="PI" value="3.141592653589793"/>
+  <material name="black">
+    <color rgba="0.0 0.0 0.0 1.0" />
+  </material>
   <!-- base -->
   <xacro:property name="base_length" value="2.695"/>
@@ -39,4 +42,7 @@
         <!-- <mesh filename="package://carmodel/meshes/vehicle_body.dae"/> -->
       </geometry>
+      <material name="yellow">
+        <color rgba="0.5 0.3 0.0 0.5" />
+      </material>
     </visual>
   </link>
